Commit message: fix(sim): harden Gazebo grasp execution and benchmark metrics

File: workspaces/app_ws/src/foam_grasp_sim/urdf/piper_eye_in_hand_gazebo.xacro (robot description, xacro)
@@ -55,4 +55,43 @@
     <origin xyz="0 0 0" rpy="-1.57079632679 0 -1.57079632679"/>
   </joint>
+  <!-- Explicit ODE contact settings for both Piper finger collision meshes. -->
+  <gazebo reference="link7">
+    <mu1>1.0</mu1>
+    <mu2>1.0</mu2>
+    <maxVel>0.01</maxVel>
+    <minDepth>0.001</minDepth>
+    <sensor name="link7_contact_sensor" type="contact">
+      <update_rate>100</update_rate>
+      <contact>
+        <collision>link7_collision</collision>
+      </contact>
+      <plugin name="link7_contact_plugin" filename="libgazebo_ros_bumper.so">
+        <ros>
+          <namespace>/foam_grasp_sim</namespace>
+          <remapping>bumper_states:=link7_contacts</remapping>
+        </ros>
+        <frame_name>link7</frame_name>
+      </plugin>
+    </sensor>
+  </gazebo>
+  <gazebo reference="link8">
+    <mu1>1.0</mu1>
+    <mu2>1.0</mu2>
+    <maxVel>0.01</maxVel>
+    <minDepth>0.001</minDepth>
+    <sensor name="link8_contact_sensor" type="contact">
+      <update_rate>100</update_rate>
+      <contact>
+        <collision>link8_collision</collision>
+      </contact>
+      <plugin name="link8_contact_plugin" filename="libgazebo_ros_bumper.so">
+        <ros>
+          <namespace>/foam_grasp_sim</namespace>
+          <remapping>bumper_states:=link8_contacts</remapping>
+        </ros>
+        <frame_name>link8</frame_name>
+      </plugin>
+    </sensor>
+  </gazebo>
   <gazebo reference="camera_link">
     <sensor name="eye_in_hand_rgbd" type="depth">

Commit message: fix(sim): calibrate eye-in-hand RGB-D pipeline

File: workspaces/app_ws/src/foam_grasp_sim/urdf/piper_eye_in_hand_gazebo.xacro (robot description, xacro)
@@ -33,5 +33,9 @@
     <parent link="link6"/>
     <child link="camera_link"/>
-    <origin xyz="0 0 0.055" rpy="0 -1.57079632679 0"/>
+    <!-- Derived from runtime/calibration/handeye_eye_in_hand.json:
+         T_link6_camera_link = T_link6_camera_optical
+           * inv(T_camera_link_camera_color_optical_frame). -->
+    <origin xyz="-0.0774037255 0.0095206804 0.0301674851"
+            rpy="0.002600958 -1.211791754 -0.037610506"/>
   </joint>
   <joint name="camera_color_frame_joint" type="fixed">
@@ -97,11 +101,13 @@
     <sensor name="eye_in_hand_rgbd" type="depth">
       <pose>0 0 0 0 0 0</pose>
-      <update_rate>15</update_rate>
+      <!-- DaBai DC1 project-validated profile: 640x480 at 30 Hz. -->
+      <update_rate>30</update_rate>
       <visualize>false</visualize>
       <camera name="eye_in_hand_rgbd">
-        <horizontal_fov>1.0472</horizontal_fov>
+        <!-- Derived from the project-validated DC1 depth fx ~= 489.48 px. -->
+        <horizontal_fov>1.158020831</horizontal_fov>
         <image>
           <width>640</width>
-          <height>360</height>
+          <height>480</height>
           <format>R8G8B8</format>
         </image>
